File: soph68.kicad_pcb (KiCad board)
At the start: 2 copper layers, 328.6 x 100.9 mm, 235 parts, among them J1 STLINK_6_Pin, U1 SRV05-4, U2 STM32F072C8Tx, U3 AMS1117-5.0

Commit message: fixing some schema troubles
Parts:
- added G***: nicole_x_silk, soph68:nicole_x_silk, B.Cu at (115.6, 133.6)
- added G***: nicole_x_silk, soph68:nicole_x_silk, F.Cu at (115.6, 133.5)
- added G***: LOGO, soph68:nicole_x_cu, F.Cu at (115.6, 133.5)
Connections:
- CSI1 pad 1: Net-(CSI1-Pad1) -> +5V
- DF1 pad 1: Net-(CSI1-Pad1) -> +5V
- DS1 pad 1: Net-(CSI1-Pad1) -> +5V
- F1 pad 1: Net-(CSI1-Pad1) -> +5V
- K_0 pad 4: VBUS -> +5V
- K_1 pad 4: VBUS -> +5V
- K_10 pad 4: VBUS -> +5V
- K_11 pad 4: VBUS -> +5V
- K_12 pad 4: VBUS -> +5V
- K_13 pad 4: VBUS -> +5V
- K_14 pad 4: VBUS -> +5V
- K_15 pad 4: VBUS -> +5V
- K_16 pad 4: VBUS -> +5V
- K_17 pad 4: VBUS -> +5V
- K_18 pad 4: VBUS -> +5V
- K_19 pad 4: VBUS -> +5V
- K_2 pad 4: VBUS -> +5V
- K_20 pad 4: VBUS -> +5V
- K_21 pad 4: VBUS -> +5V
- K_22 pad 4: VBUS -> +5V
- K_23 pad 4: VBUS -> +5V
- K_24 pad 4: VBUS -> +5V
- K_25 pad 4: VBUS -> +5V
- K_26 pad 4: VBUS -> +5V
- K_27 pad 4: VBUS -> +5V
- K_28 pad 4: VBUS -> +5V
- K_29 pad 4: VBUS -> +5V
- K_3 pad 4: VBUS -> +5V
- K_30 pad 4: VBUS -> +5V
- K_31 pad 4: VBUS -> +5V
- K_32 pad 4: VBUS -> +5V
- K_33 pad 4: VBUS -> +5V
- K_34 pad 4: VBUS -> +5V
- K_35 pad 4: VBUS -> +5V
- K_36 pad 4: VBUS -> +5V
- K_37 pad 4: VBUS -> +5V
- K_38 pad 4: VBUS -> +5V
- K_39 pad 4: VBUS -> +5V
- K_4 pad 4: VBUS -> +5V
- K_40 pad 4: VBUS -> +5V
- K_41 pad 4: VBUS -> +5V
- K_42 pad 4: VBUS -> +5V
- K_43 pad 4: VBUS -> +5V
- K_44 pad 4: VBUS -> +5V
- K_45 pad 4: VBUS -> +5V
- K_46 pad 4: VBUS -> +5V
- K_47 pad 4: VBUS -> +5V
- K_48 pad 4: VBUS -> +5V
- K_49 pad 4: VBUS -> +5V
- K_5 pad 4: VBUS -> +5V
- K_50 pad 4: VBUS -> +5V
- K_51 pad 4: VBUS -> +5V
- K_52 pad 4: VBUS -> +5V
- K_53 pad 4: VBUS -> +5V
- K_54 pad 4: VBUS -> +5V
- K_55 pad 4: VBUS -> +5V
- K_56 pad 4: VBUS -> +5V
- K_57 pad 4: VBUS -> +5V
- K_58 pad 4: VBUS -> +5V
- K_59 pad 4: VBUS -> +5V
- K_6 pad 4: VBUS -> +5V
- K_60 pad 4: VBUS -> +5V
- K_61 pad 4: VBUS -> +5V
- K_62 pad 4: VBUS -> +5V
- K_63 pad 4: VBUS -> +5V
- K_64 pad 4: VBUS -> +5V
- K_65 pad 4: VBUS -> +5V
- K_66 pad 4: VBUS -> +5V
- K_67 pad 4: VBUS -> +5V
- K_7 pad 4: VBUS -> +5V
- K_8 pad 4: VBUS -> +5V
- K_9 pad 4: VBUS -> +5V
- RCC1 pad 1: Net-(RCC1-Pad1) -> GND
- RCC2 pad 1: Net-(RCC2-Pad1) -> GND
- RSI1 pad 1: Net-(CSI1-Pad1) -> +5V
- U3 pad 3: Net-(CSI1-Pad1) -> +5V
Routing:
- net +5V: track 0.00 -> 1760.7 mm, vias 0 -> 2
- net VBUS: track 1787.8 -> 48.8 mm, vias 2 -> 0
- net Net-(CSI1-Pad1): track 17.0 -> 0.00 mm
Other:
- board text added: "nicole aptekar"
- board text added: "soph68 v1"

Commit message: Rerouted things to get rid of 45s
Routing:
- net row1: track 379.7 -> 362.0 mm
- net row2: track 323.6 -> 309.2 mm
- net LED-: track 1698.5 -> 1685.5 mm
- net row0: track 392.3 -> 381.0 mm
- net row3: track 311.7 -> 301.4 mm
- net +5V: track 1760.7 -> 1755.7 mm
- net row4: track 357.4 -> 354.8 mm
- net Net-(CSH1-Pad2): track 27.5 -> 28.8 mm
- net GND: vias 66 -> 64

Commit message: Changed vias a bit
Routing:
- net GND: vias 64 -> 54
Changed lines of the file:
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@@
     (thickness 1.6)
     (drawings 16)
-    (tracks 1965)
+    (tracks 1955)
     (zones 0)
     (modules 238)
@@
   )
   (module MX_Only:MXOnly-1U (layer F.Cu)
+    (at 219.075 95.25)
+    (fp_text reference K_41 (at 0 3.175) (layer Dwgs.User)
+      (effects (font (size 1 1) (thickness 0.15)))
+    )
+    (fp_text value KEYSW (at 0 -7.9375) (layer Dwgs.User)
+      (effects (font (size 1 1) (thickness 0.15)))
+    )
+    (fp_line (start -9.525 9.525) (end -9.525 -9.525) (layer Dwgs.User) (width 0.15))
+    (fp_line (start 9.525 9.525) (end -9.525 9.525) (layer Dwgs.User) (width 0.15))
+    (fp_line (start 9.525 -9.525) (end 9.525 9.525) (layer Dwgs.User) (width 0.15))
+    (fp_line (start -9.525 -9.525) (end 9.525 -9.525) (layer Dwgs.User) (width 0.15))
+    (fp_line (start -7 -7) (end -7 -5) (layer Dwgs.User) (width 0.15))
+    (fp_line (start -5 -7) (end -7 -7) (layer Dwgs.User) (width 0.15))
+    (fp_line (start -7 7) (end -5 7) (layer Dwgs.User) (width 0.15))
+    (fp_line (start -7 5) (end -7 7) (layer Dwgs.User) (width 0.15))
+    (fp_line (start 7 7) (end 7 5) (layer Dwgs.User) (width 0.15))
+    (fp_line (start 5 7) (end 7 7) (layer Dwgs.User) (width 0.15))
+    (fp_line (start 7 -7) (end 7 -5) (layer Dwgs.User) (width 0.15))
+    (fp_line (start 5 -7) (end 7 -7) (layer Dwgs.User) (width 0.15))
+    (pad "" np_thru_hole circle (at 5.08 0 48.0996) (size 1.75 1.75) (drill 1.75) (layers *.Cu *.Mask))
+    (pad "" np_thru_hole circle (at -5.08 0 48.0996) (size 1.75 1.75) (drill 1.75) (layers *.Cu *.Mask))
+    (pad 4 thru_hole rect (at 1.27 5.08) (size 1.905 1.905) (drill 1.04) (layers *.Cu B.Mask)
+      (net 189 +5V))
+    (pad 3 thru_hole circle (at -1.27 5.08) (size 1.905 1.905) (drill 1.04) (layers *.Cu B.Mask)
+      (net 106 "Net-(K_41-Pad3)"))
+    (pad 1 thru_hole circle (at -3.81 -2.54) (size 2.25 2.25) (drill 1.47) (layers *.Cu B.Mask)
+      (net 12 col10))
+    (pad "" np_thru_hole circle (at 0 0) (size 3.9878 3.9878) (drill 3.9878) (layers *.Cu *.Mask))
+    (pad 2 thru_hole circle (at 2.54 -5.08) (size 2.25 2.25) (drill 1.47) (layers *.Cu B.Mask)
+      (net 107 "Net-(D_41-Pad2)"))
+  )
+  (module MX_Only:MXOnly-1U (layer F.Cu)
     (at 252.4125 76.2)
     (fp_text reference K_27 (at 0 3.175) (layer Dwgs.User)
@@
   )
   (module MX_Only:MXOnly-1U (layer F.Cu)
-    (at 219.075 95.25)
-    (fp_text reference K_41 (at 0 3.175) (layer Dwgs.User)
-      (effects (font (size 1 1) (thickness 0.15)))
-    )
-    (fp_text value KEYSW (at 0 -7.9375) (layer Dwgs.User)
-      (effects (font (size 1 1) (thickness 0.15)))
-    )
-    (fp_line (start -9.525 9.525) (end -9.525 -9.525) (layer Dwgs.User) (width 0.15))
-    (fp_line (start 9.525 9.525) (end -9.525 9.525) (layer Dwgs.User) (width 0.15))
-    (fp_line (start 9.525 -9.525) (end 9.525 9.525) (layer Dwgs.User) (width 0.15))
-    (fp_line (start -9.525 -9.525) (end 9.525 -9.525) (layer Dwgs.User) (width 0.15))
-    (fp_line (start -7 -7) (end -7 -5) (layer Dwgs.User) (width 0.15))
-    (fp_line (start -5 -7) (end -7 -7) (layer Dwgs.User) (width 0.15))
-    (fp_line (start -7 7) (end -5 7) (layer Dwgs.User) (width 0.15))
-    (fp_line (start -7 5) (end -7 7) (layer Dwgs.User) (width 0.15))
-    (fp_line (start 7 7) (end 7 5) (layer Dwgs.User) (width 0.15))
-    (fp_line (start 5 7) (end 7 7) (layer Dwgs.User) (width 0.15))
-    (fp_line (start 7 -7) (end 7 -5) (layer Dwgs.User) (width 0.15))
-    (fp_line (start 5 -7) (end 7 -7) (layer Dwgs.User) (width 0.15))
-    (pad "" np_thru_hole circle (at 5.08 0 48.0996) (size 1.75 1.75) (drill 1.75) (layers *.Cu *.Mask))
-    (pad "" np_thru_hole circle (at -5.08 0 48.0996) (size 1.75 1.75) (drill 1.75) (layers *.Cu *.Mask))
-    (pad 4 thru_hole rect (at 1.27 5.08) (size 1.905 1.905) (drill 1.04) (layers *.Cu B.Mask)
-      (net 189 +5V))
-    (pad 3 thru_hole circle (at -1.27 5.08) (size 1.905 1.905) (drill 1.04) (layers *.Cu B.Mask)
-      (net 106 "Net-(K_41-Pad3)"))
-    (pad 1 thru_hole circle (at -3.81 -2.54) (size 2.25 2.25) (drill 1.47) (layers *.Cu B.Mask)
-      (net 12 col10))
-    (pad "" np_thru_hole circle (at 0 0) (size 3.9878 3.9878) (drill 3.9878) (layers *.Cu *.Mask))
-    (pad 2 thru_hole circle (at 2.54 -5.08) (size 2.25 2.25) (drill 1.47) (layers *.Cu B.Mask)
-      (net 107 "Net-(D_41-Pad2)"))
-  )
-  (module MX_Only:MXOnly-1U (layer F.Cu)
     (at 200.025 95.25)
     (fp_text reference K_40 (at 0 3.175) (layer Dwgs.User)
@@
   (segment (start 308.883 48.307) (end 308.883 49.657) (width 0.25) (layer B.Cu) (net 1))
   (via (at 308.356 100.076) (size 0.8) (drill 0.4) (layers F.Cu B.Cu) (net 1))
-  (via (at 304.038 92.583) (size 0.8) (drill 0.4) (layers F.Cu B.Cu) (net 1))
   (via (at 279.908 88.138) (size 0.8) (drill 0.4) (layers F.Cu B.Cu) (net 1))
   (via (at 275.0185 64.5795) (size 0.8) (drill 0.4) (layers F.Cu B.Cu) (net 1))
@@
   (via (at 80.9625 62.23) (size 0.8) (drill 0.4) (layers F.Cu B.Cu) (net 1))
   (via (at 61.9125 62.23) (size 0.8) (drill 0.4) (layers F.Cu B.Cu) (net 1))
-  (via (at 71.501 81.28) (size 0.8) (drill 0.4) (layers F.Cu B.Cu) (net 1))
-  (via (at 52.451 81.153) (size 0.8) (drill 0.4) (layers F.Cu B.Cu) (net 1))
   (via (at 90.551 81.28) (size 0.8) (drill 0.4) (layers F.Cu B.Cu) (net 1))
   (via (at 109.474 81.407) (size 0.8) (drill 0.4) (layers F.Cu B.Cu) (net 1))
@@
   (via (at 42.926 73.533) (size 0.8) (drill 0.4) (layers F.Cu B.Cu) (net 1))
   (via (at 162.433 73.533) (size 0.8) (drill 0.4) (layers F.Cu B.Cu) (net 1))
-  (via (at 57.277 100.203) (size 0.8) (drill 0.4) (layers F.Cu B.Cu) (net 1))
-  (via (at 76.327 100.33) (size 0.8) (drill 0.4) (layers F.Cu B.Cu) (net 1))
-  (via (at 95.25 100.33) (size 0.8) (drill 0.4) (layers F.Cu B.Cu) (net 1))
-  (via (at 114.3 100.203) (size 0.8) (drill 0.4) (layers F.Cu B.Cu) (net 1))
-  (via (at 133.35 100.203) (size 0.8) (drill 0.4) (layers F.Cu B.Cu) (net 1))
-  (via (at 152.4 100.203) (size 0.8) (drill 0.4) (layers F.Cu B.Cu) (net 1))
-  (via (at 171.45 100.457) (size 0.8) (drill 0.4) (layers F.Cu B.Cu) (net 1))
-  (via (at 190.627 100.457) (size 0.8) (drill 0.4) (layers F.Cu B.Cu) (net 1))
-  (via (at 209.55 100.33) (size 0.8) (drill 0.4) (layers F.Cu B.Cu) (net 1))
-  (via (at 228.6 100.33) (size 0.8) (drill 0.4) (layers F.Cu B.Cu) (net 1))
-  (via (at 247.65 100.33) (size 0.8) (drill 0.4) (layers F.Cu B.Cu) (net 1))
-  (via (at 238.125 119.507) (size 0.8) (drill 0.4) (layers F.Cu B.Cu) (net 1))
-  (via (at 218.948 119.507) (size 0.8) (drill 0.4) (layers F.Cu B.Cu) (net 1))
-  (via (at 200.025 119.38) (size 0.8) (drill 0.4) (layers F.Cu B.Cu) (net 1))
-  (via (at 180.975 119.38) (size 0.8) (drill 0.4) (layers F.Cu B.Cu) (net 1))
-  (via (at 161.925 119.38) (size 0.8) (drill 0.4) (layers F.Cu B.Cu) (net 1))
-  (via (at 142.875 119.253) (size 0.8) (drill 0.4) (layers F.Cu B.Cu) (net 1))
-  (via (at 123.825 119.38) (size 0.8) (drill 0.4) (layers F.Cu B.Cu) (net 1))
-  (via (at 47.625 138.557) (size 0.8) (drill 0.4) (layers F.Cu B.Cu) (net 1))
-  (via (at 71.374 138.557) (size 0.8) (drill 0.4) (layers F.Cu B.Cu) (net 1))
-  (via (at 95.25 138.557) (size 0.8) (drill 0.4) (layers F.Cu B.Cu) (net 1))
-  (via (at 169.418 138.43) (size 0.8) (drill 0.4) (layers F.Cu B.Cu) (net 1))
-  (via (at 237.998 138.303) (size 0.8) (drill 0.4) (layers F.Cu B.Cu) (net 1))
-  (via (at 262.001 138.557) (size 0.8) (drill 0.4) (layers F.Cu B.Cu) (net 1))
-  (via (at 285.877 138.303) (size 0.8) (drill 0.4) (layers F.Cu B.Cu) (net 1))
   (via (at 285.623 127.635) (size 0.8) (drill 0.4) (layers F.Cu B.Cu) (net 1))
-  (via (at 314.325 138.43) (size 0.8) (drill 0.4) (layers F.Cu B.Cu) (net 1))
   (via (at 314.325 127.889) (size 0.8) (drill 0.4) (layers F.Cu B.Cu) (net 1))
-  (via (at 257.175 119.507) (size 0.8) (drill 0.4) (layers F.Cu B.Cu) (net 1))
   (via (at 333.375 74.93) (size 0.8) (drill 0.4) (layers F.Cu B.Cu) (net 1))
   (via (at 333.375 66.421) (size 0.8) (drill 0.4) (layers F.Cu B.Cu) (net 1))
@@
   (via (at 42.8625 62.1665) (size 0.8) (drill 0.4) (layers F.Cu B.Cu) (net 1))
   (via (at 252.4125 62.1665) (size 0.8) (drill 0.4) (layers F.Cu B.Cu) (net 1))
+  (via (at 302.768 91.567) (size 0.8) (drill 0.4) (layers F.Cu B.Cu) (net 1))
+  (via (at 336.296 115.824) (size 0.8) (drill 0.4) (layers F.Cu B.Cu) (net 1))
+  (via (at 344.043 118.491) (size 0.8) (drill 0.4) (layers F.Cu B.Cu) (net 1))
+  (via (at 157.353 54.737) (size 0.8) (drill 0.4) (layers F.Cu B.Cu) (net 1))
+  (via (at 153.924 92.456) (size 0.8) (drill 0.4) (layers F.Cu B.Cu) (net 1))
+  (via (at 154.686 103.378) (size 0.8) (drill 0.4) (layers F.Cu B.Cu) (net 1))
+  (via (at 161.29 112.522) (size 0.8) (drill 0.4) (layers F.Cu B.Cu) (net 1))
+  (via (at 159.385 122.936) (size 0.8) (drill 0.4) (layers F.Cu B.Cu) (net 1))
+  (via (at 164.338 131.826) (size 0.8) (drill 0.4) (layers F.Cu B.Cu) (net 1))
+  (via (at 274.066 56.515) (size 0.8) (drill 0.4) (layers F.Cu B.Cu) (net 1))
+  (via (at 276.098 94.615) (size 0.8) (drill 0.4) (layers F.Cu B.Cu) (net 1))
+  (via (at 273.812 114.3) (size 0.8) (drill 0.4) (layers F.Cu B.Cu) (net 1))
+  (via (at 283.591 133.731) (size 0.8) (drill 0.4) (layers F.Cu B.Cu) (net 1))
+  (via (at 282.321 140.335) (size 0.8) (drill 0.4) (layers F.Cu B.Cu) (net 1))
+  (via (at 44.069 85.852) (size 0.8) (drill 0.4) (layers F.Cu B.Cu) (net 1))
+  (via (at 42.799 54.737) (size 0.8) (drill 0.4) (layers F.Cu B.Cu) (net 1))
+  (via (at 44.069 105.029) (size 0.8) (drill 0.4) (layers F.Cu B.Cu) (net 1))
+  (via (at 44.069 123.571) (size 0.8) (drill 0.4) (layers F.Cu B.Cu) (net 1))
+  (via (at 44.196 132.207) (size 0.8) (drill 0.4) (layers F.Cu B.Cu) (net 1))
+  (via (at 44.196 140.589) (size 0.8) (drill 0.4) (layers F.Cu B.Cu) (net 1))
   (segment (start 29.5275 68.8975) (end 34.29 73.66) (width 0.25) (layer F.Cu) (net 2))
   (segment (start 34.29 90.32875) (end 36.67125 92.71) (width 0.25) (layer F.Cu) (net 2))
