File: soph68.kicad_pcb (KiCad board)
At the start: 2 copper layers, 328.6 x 100.9 mm, 238 parts, among them J1 STLINK_6_Pin, U1 SRV05-4, U2 STM32F072C8Tx, U3 AMS1117-5.0

Commit message: Changed to cbtx
Parts:
- U2: value STM32F072C8Tx -> STM32F072CBTx
Changed lines of the file:
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@@
     (35 F.Paste user)
     (36 B.SilkS user)
-    (37 F.SilkS user)
+    (37 F.SilkS user hide)
     (38 B.Mask user)
     (39 F.Mask user)
@@
     (tags "SPST Button Switch")
     (attr smd)
-    (fp_text reference SWRST1 (at 0 3.6) (layer B.SilkS)
+    (fp_text reference SWRST1 (at 0 -3.683) (layer B.SilkS)
       (effects (font (size 1 1) (thickness 0.15)) (justify mirror))
     )
@@
     (tags capacitor)
     (attr smd)
-    (fp_text reference CBT1 (at 0 1.17) (layer B.SilkS)
-      (effects (font (size 1 1) (thickness 0.15)) (justify mirror))
+    (fp_text reference CBT1 (at 1.905 0) (layer B.SilkS)
+      (effects (font (size 0.5 0.5) (thickness 0.1)) (justify mirror))
     )
     (fp_text value 100nF (at 0 -1.17) (layer B.Fab)
@@
     (tags capacitor)
     (attr smd)
-    (fp_text reference RSI1 (at 0 1.65 90) (layer B.SilkS)
+    (fp_text reference RSI1 (at -2.413 0.254 180) (layer B.SilkS)
       (effects (font (size 1 1) (thickness 0.15)) (justify mirror))
     )
@@
     (tags resistor)
     (attr smd)
-    (fp_text reference F1 (at 0 2.65 90) (layer B.SilkS)
+    (fp_text reference F1 (at 3.556 0 180) (layer B.SilkS)
       (effects (font (size 1 1) (thickness 0.15)) (justify mirror))
     )
@@
     (tags "Diode SMB (DO-214AA)")
     (attr smd)
-    (fp_text reference DF1 (at 0 3 90) (layer B.SilkS)
+    (fp_text reference DF1 (at 4.2545 0 180) (layer B.SilkS)
       (effects (font (size 1 1) (thickness 0.15)) (justify mirror))
     )
@@
     (tags "Diode MELF ")
     (attr smd)
-    (fp_text reference DS1 (at 0 2.5 90) (layer B.SilkS)
+    (fp_text reference DS1 (at 2.0955 2.413 90) (layer B.SilkS)
       (effects (font (size 1 1) (thickness 0.15)) (justify mirror))
     )
@@
     (tags capacitor)
     (attr smd)
-    (fp_text reference CSO1 (at 0 1.65 90) (layer B.SilkS)
-      (effects (font (size 1 1) (thickness 0.15)) (justify mirror))
+    (fp_text reference CSO1 (at -2.032 0 180) (layer B.SilkS)
+      (effects (font (size 0.5 0.5) (thickness 0.1)) (justify mirror))
     )
     (fp_text value 1u (at 0 -1.65 90) (layer B.Fab)
@@
     (tags capacitor)
     (attr smd)
-    (fp_text reference CSI1 (at 0 1.65 90) (layer B.SilkS)
-      (effects (font (size 1 1) (thickness 0.15)) (justify mirror))
+    (fp_text reference CSI1 (at -2.159 0 180) (layer B.SilkS)
+      (effects (font (size 0.5 0.5) (thickness 0.1)) (justify mirror))
     )
     (fp_text value 1u (at 0 -1.65 90) (layer B.Fab)
@@
     (tags resistor)
     (attr smd)
-    (fp_text reference RSH1 (at 0 1.65 90) (layer B.SilkS)
-      (effects (font (size 1 1) (thickness 0.15)) (justify mirror))
+    (fp_text reference RSH1 (at 2.159 0 180) (layer B.SilkS)
+      (effects (font (size 0.5 0.5) (thickness 0.1)) (justify mirror))
     )
     (fp_text value 1M (at 0 -1.65 90) (layer B.Fab)
@@
     (tags capacitor)
     (attr smd)
-    (fp_text reference CSH1 (at 0 1.65 90) (layer B.SilkS)
-      (effects (font (size 1 1) (thickness 0.15)) (justify mirror))
+    (fp_text reference CSH1 (at 2.159 0 180) (layer B.SilkS)
+      (effects (font (size 0.5 0.5) (thickness 0.1)) (justify mirror))
     )
     (fp_text value 4.7nF (at 0 -1.65 90) (layer B.Fab)
@@
       (effects (font (size 1 1) (thickness 0.15)) (justify mirror))
     )
-    (fp_text value STM32F072C8Tx (at 0 -5.85 135) (layer B.Fab)
+    (fp_text value STM32F072CBTx (at 0 -5.85 135) (layer B.Fab)
       (effects (font (size 1 1) (thickness 0.15)) (justify mirror))
     )
@@
     (tags resistor)
     (attr smd)
-    (fp_text reference RBT1 (at 0 1.65) (layer B.SilkS)
-      (effects (font (size 1 1) (thickness 0.15)) (justify mirror))
+    (fp_text reference RBT1 (at 0 -1.27) (layer B.SilkS)
+      (effects (font (size 0.5 0.5) (thickness 0.1)) (justify mirror))
     )
     (fp_text value 10k (at 0 -1.65) (layer B.Fab)
@@
     (tags resistor)
     (attr smd)
-    (fp_text reference RLED1 (at 0 1.17) (layer B.SilkS)
+    (fp_text reference RLED1 (at -3.2385 0) (layer B.SilkS)
       (effects (font (size 1 1) (thickness 0.15)) (justify mirror))
     )
@@
     (tags SOT-23)
     (attr smd)
-    (fp_text reference QLED1 (at 0 2.5 90) (layer B.SilkS)
+    (fp_text reference QLED1 (at 2.3495 0 180) (layer B.SilkS)
       (effects (font (size 1 1) (thickness 0.15)) (justify mirror))
     )
@@
     (tags capacitor)
     (attr smd)
-    (fp_text reference CRST1 (at 0 1.17) (layer B.SilkS)
-      (effects (font (size 1 1) (thickness 0.15)) (justify mirror))
+    (fp_text reference CRST1 (at 2.159 0) (layer B.SilkS)
+      (effects (font (size 0.5 0.5) (thickness 0.1)) (justify mirror))
     )
     (fp_text value 100nF (at 0 -1.17) (layer B.Fab)
@@
     (tags capacitor)
     (attr smd)
-    (fp_text reference CB8 (at 0 1.17 45) (layer B.SilkS)
-      (effects (font (size 1 1) (thickness 0.15)) (justify mirror))
+    (fp_text reference CB8 (at 1.706249 -0.089803 45) (layer B.SilkS)
+      (effects (font (size 0.5 0.5) (thickness 0.1)) (justify mirror))
     )
     (fp_text value 4.7uF (at 0 -1.17 45) (layer B.Fab)
@@
     (tags capacitor)
     (attr smd)
-    (fp_text reference CB7 (at 0 1.17 45) (layer B.SilkS)
-      (effects (font (size 1 1) (thickness 0.15)) (justify mirror))
+    (fp_text reference CB7 (at 1.706249 -0.089803 45) (layer B.SilkS)
+      (effects (font (size 0.5 0.5) (thickness 0.1)) (justify mirror))
     )
     (fp_text value 100nF (at 0 -1.17 45) (layer B.Fab)
@@
     (tags capacitor)
     (attr smd)
-    (fp_text reference CB6 (at 0 1.17) (layer B.SilkS)
-      (effects (font (size 1 1) (thickness 0.15)) (justify mirror))
+    (fp_text reference CB6 (at 1.674 0) (layer B.SilkS)
+      (effects (font (size 0.5 0.5) (thickness 0.1)) (justify mirror))
     )
     (fp_text value 1uF (at 0 -1.17) (layer B.Fab)
@@
     (tags capacitor)
     (attr smd)
-    (fp_text reference CB5 (at 0 1.17) (layer B.SilkS)
-      (effects (font (size 1 1) (thickness 0.15)) (justify mirror))
+    (fp_text reference CB5 (at 1.705 -0.01925) (layer B.SilkS)
+      (effects (font (size 0.5 0.5) (thickness 0.1)) (justify mirror))
     )
     (fp_text value 10n (at 0 -1.17) (layer B.Fab)
@@
     (tags capacitor)
     (attr smd)
-    (fp_text reference CB3 (at 0 1.17) (layer B.SilkS)
-      (effects (font (size 1 1) (thickness 0.15)) (justify mirror))
+    (fp_text reference CB3 (at 1.778 0) (layer B.SilkS)
+      (effects (font (size 0.5 0.5) (thickness 0.1)) (justify mirror))
     )
     (fp_text value 4.7uF (at 0 -1.17) (layer B.Fab)
@@
     (tags capacitor)
     (attr smd)
-    (fp_text reference CB2 (at 0 1.17) (layer B.SilkS)
-      (effects (font (size 1 1) (thickness 0.15)) (justify mirror))
+    (fp_text reference CB2 (at 1.778 0) (layer B.SilkS)
+      (effects (font (size 0.5 0.5) (thickness 0.1)) (justify mirror))
     )
     (fp_text value 100nF (at 0 -1.17) (layer B.Fab)
